File: pragotron-clock.kicad_sch (KiCad schematic)
At the start: 8 parts, among them J1 Conn_01x02, J2 Conn_01x03, J3 Conn_01x03, U1 L293D, U2 ESP32_DEVCITV1

Commit message: control schematic
Parts:
- added C1: 10u 100V MLCC, Capacitor_THT:C_Rect_L7.0mm_W3.5mm_P5.00mm, symbol Device:C
- added J4: Conn_01x02, Connector_JST:JST_XH_S2B-XH-A-1_1x02_P2.50mm_Horizontal, symbol Connector_Generic:Conn_01x02
- added PS1: ROE-2405S, JS_Local:ROE1205S, symbol JS_Local:ROE-2405S
- J1: footprint (none) -> Connector_JST:JST_XH_S2B-XH-A-1_1x02_P2.50mm_Horizontal
- J2, J3: footprint (none) -> Connector_JST:JST_XH_S3B-XH-A-1_1x03_P2.50mm_Horizontal
- R1, R2, R3: footprint (none) -> Resistor_THT:R_Axial_DIN0204_L3.6mm_D1.6mm_P7.62mm_Horizontal
Connections:
- net +24V: now also C1.1, J4.1 (Pin_1), PS1.2 (+VIN)
- net +5V: now also U2.15 (VIN), PS1.4 (+VOUT); no longer U1.16 (VCC1)
- net GND: now also U1.12 (GND), U1.13 (GND), U1.4 (GND), U1.5 (GND), U1.9 (EN3,4), C1.2, J4.2 (Pin_2), PS1.1 (-VIN), PS1.3 (-VOUT)
- net at J2.1 (Pin_1), J3.1 (Pin_1), R2.2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: now also U1.16 (VCC1)
- no-connect marks 0 -> 4
