File: pcb/pragotron-clock.kicad_sch (KiCad schematic)
At the start: 11 parts, among them J1 Conn_01x02, J2 Conn_01x03, J3 Conn_01x03, J4 Conn_01x02, U1 L293D, U2 ESP32_DEVCITV1

Commit message: schematics+
Parts:
- removed U2: ESP32_DEVCITV1, JS_Local:ESP32_DEVKITV1, symbol JS_Local:ESP32_DEVCITV1
- added C2, C3: 100n, symbol Device:C
- added F1, F2: Fuse, symbol Device:Fuse
- added J5: Conn_01x02, Connector_JST:JST_XH_S2B-XH-A-1_1x02_P2.50mm_Horizontal, symbol Connector_Generic:Conn_01x02
- added J6: Conn_01x04, symbol Connector_Generic:Conn_01x04
- added U2: ~, symbol JS_Local:ESP8266_12E_DEVKIT
Connections:
- net +5V: now also C3.1, U2. (3V3)
- net GND: now also C2.2, C3.2, J6.2 (Pin_2), J6.4 (Pin_4), U2. (3V3)
- net +3V3: now reaches R1.1, U1.1 (EN1,2)
- net +3V3: now also J2.1 (Pin_1), J3.1 (Pin_1), R2.2, R3.1, U1.16 (VCC1), C2.1, J6.1 (Pin_1), U2. (3V3)
- net at U1.11 (3Y): now also F2.1
- net at U1.14 (4Y): now also J5.2 (Pin_2)
- net at U1.2 (1A): now also U2. (3V3)
- net at U1.3 (1Y): now also F1.1; no longer J1.1 (Pin_1)
- net at U1.7 (2A): now also U2. (3V3)
- net at J2.3 (Pin_3), R2.1: now also U2. (3V3)
- net at J3.3 (Pin_3), R3.2: now also U2. (3V3)
- new net: F2.2, J5.1 (Pin_1)
- new net: F1.2, J1.1 (Pin_1)
- new net: J6.3 (Pin_3), U2. (3V3)
- no-connect marks 4 -> 2
Other:
- note added: "EN"
- note added: "GND"
- note added: "SIGNAL"
- note added: "VCC"
- moved on the sheet: J1

Commit message: wip firmware and schematics
Parts:
- removed R1: 47K, Resistor_THT:R_Axial_DIN0204_L3.6mm_D1.6mm_P7.62mm_Horizontal, symbol Device:R
- U2: value ~ -> (none)
Connections:
- net +3V3: now also U1.9 (EN3,4)
- net +5V: no longer C3.1
- net GND: no longer U1.9 (EN3,4)
- net OUT2_POSITIVE: now reaches U1.10 (3A)
- net OUT2_POSITIVE: now also U2. (3V3)
- net OUT2_NEGATIVE: now reaches U1.15 (4A)
- net OUT2_NEGATIVE: now also U2. (3V3)
- net OUT1_POSITIVE: now reaches U1.2 (1A), U2. (3V3)
- net OUT1_NEGATIVE: now reaches U1.7 (2A), U2. (3V3)
- net SENS1: now reaches J3.3 (Pin_3), R3.2, U2. (3V3)
- net DCF_SIG: now reaches J6.3 (Pin_3), U2. (3V3)
- net SENS2: now reaches J2.3 (Pin_3), R2.1, U2. (3V3)
- new net: C3.1, U2. (3V3)
- no-connect marks 2 -> 0
Other:
- moved on the sheet: C2, C3, J2, J3, R2, R3

Commit message: schematic
Parts:
- removed J4: Conn_01x02, Connector_JST:JST_XH_S2B-XH-A-1_1x02_P2.50mm_Horizontal, symbol Connector_Generic:Conn_01x02
- added J7: 694108301002, JS_Local:694108301002, symbol JS_Local:694108301002
- C2, C3: footprint (none) -> Capacitor_SMD:C_1206_3216Metric_Pad1.33x1.80mm_HandSolder
- F1, F2: footprint (none) -> Fuse:Fuse_1206_3216Metric_Pad1.42x1.75mm_HandSolder
- J6: footprint (none) -> JS_Local:DCF77
- R2, R3: footprint Resistor_THT:R_Axial_DIN0204_L3.6mm_D1.6mm_P7.62mm_Horizontal -> Resistor_SMD:R_1206_3216Metric_Pad1.30x1.75mm_HandSolder
- U2: footprint (none) -> JS_Local:ESP8266_12E_DEVKIT
Connections:
- net +24V: now also J7.1
- net +3V3: now also U2.15 (3V3), U2.20 (3V3), U2.6 (3V3); no longer U2. (3V3)
- net +5V: now also C3.1, U2.16 (VIN); no longer U2. (3V3)
- net DCF_SIG: now also U2.10 (D7); no longer U2. (3V3)
- net GND: now also U2.14 (GND), U2.17 (GND), U2.21 (GND), U2.7 (GND), J7.2, J7.3; no longer U2. (3V3)
- net OUT1_NEGATIVE: now also U2.4 (D3); no longer U2. (3V3)
- net OUT1_POSITIVE: now also U2.3 (D2); no longer U2. (3V3)
- net OUT2_NEGATIVE: now also U2.2 (D1); no longer U2. (3V3)
- net OUT2_POSITIVE: now also U2.1 (D0); no longer U2. (3V3)
- net SENS1: now also U2.8 (D5); no longer U2. (3V3)
- net SENS2: now also U2.9 (D6); no longer U2. (3V3)
- no-connect marks 0 -> 13

Commit message: minification
Parts:
- removed F2: Fuse, Fuse:Fuse_1206_3216Metric_Pad1.42x1.75mm_HandSolder, symbol Device:Fuse
- removed J5: Conn_01x02, Connector_JST:JST_XH_S2B-XH-A-1_1x02_P2.50mm_Horizontal, symbol Connector_Generic:Conn_01x02
Connections:
- net +3V3: no longer U1.9 (EN3,4)
- net GND: now also U1.9 (EN3,4)
- net OUT2_NEGATIVE: no longer names the net of U1.15 (4A)
- net OUT2_NEGATIVE: no longer U2.2 (D1)
- net OUT2_POSITIVE: no longer names the net of U1.10 (3A)
- net OUT2_POSITIVE: no longer U2.1 (D0)
- no-connect marks 13 -> 19
Changed lines of the file:
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@@
+	)
+	(junction
+		(at 199.39 99.06)
+		(diameter 0)
+		(color 0 0 0 0)
 	)
 	(junction
@@
 	)
 	(junction
-		(at 186.69 85.09)
-		(diameter 0)
-		(color 0 0 0 0)
-	)
-	(junction
 		(at 213.36 99.06)
 		(diameter 0)
@@
 	)
 	(no_connect
+		(at 231.14 80.01)
+	)
+	(no_connect
 		(at 147.32 68.58)
 	)
 	(no_connect
+		(at 231.14 74.93)
+	)
+	(no_connect
 		(at 127 71.12)
 	)
 	(no_connect
+		(at 147.32 60.96)
+	)
+	(no_connect
 		(at 127 88.9)
 	)
 	(no_connect
+		(at 147.32 58.42)
+	)
+	(no_connect
 		(at 127 73.66)
 	)
@@
 	)
 	(no_connect
+		(at 205.74 74.93)
+	)
+	(no_connect
 		(at 147.32 88.9)
 	)
@@
 	)
 	(no_connect
+		(at 205.74 80.01)
+	)
+	(no_connect
 		(at 147.32 83.82)
 	)
@@
 	(wire
 		(pts
+			(xy 199.39 99.06) (xy 186.69 99.06)
+		)
+		(stroke
+			(width 0)
+			(type default)
+		)
+	)
+	(wire
+		(pts
 			(xy 229.87 137.16) (xy 224.79 137.16)
 		)
@@
 	(wire
 		(pts
-			(xy 231.14 80.01) (xy 262.89 80.01)
-		)
-		(stroke
-			(width 0)
-			(type default)
-		)
-	)
-	(wire
-		(pts
 			(xy 147.32 71.12) (xy 170.18 71.12)
 		)
@@
 	(wire
 		(pts
-			(xy 250.19 74.93) (xy 262.89 74.93)
-		)
-		(stroke
-			(width 0)
-			(type default)
-		)
-	)
-	(wire
-		(pts
 			(xy 186.69 96.52) (xy 186.69 99.06)
 		)
@@
 	(wire
 		(pts
+			(xy 199.39 85.09) (xy 199.39 99.06)
+		)
+		(stroke
+			(width 0)
+			(type default)
+		)
+	)
+	(wire
+		(pts
 			(xy 213.36 95.25) (xy 213.36 99.06)
 		)
@@
 	(wire
 		(pts
-			(xy 186.69 85.09) (xy 186.69 88.9)
+			(xy 186.69 69.85) (xy 186.69 88.9)
 		)
 		(stroke
@@
 	(wire
 		(pts
+			(xy 205.74 85.09) (xy 199.39 85.09)
+		)
+		(stroke
+			(width 0)
+			(type default)
+		)
+	)
+	(wire
+		(pts
 			(xy 220.98 99.06) (xy 220.98 95.25)
 		)
@@
 	(wire
 		(pts
-			(xy 186.69 85.09) (xy 205.74 85.09)
-		)
-		(stroke
-			(width 0)
-			(type default)
-		)
-	)
-	(wire
-		(pts
-			(xy 213.36 99.06) (xy 186.69 99.06)
-		)
-		(stroke
-			(width 0)
-			(type default)
-		)
-	)
-	(wire
-		(pts
-			(xy 231.14 74.93) (xy 242.57 74.93)
-		)
-		(stroke
-			(width 0)
-			(type default)
-		)
-	)
-	(wire
-		(pts
-			(xy 186.69 85.09) (xy 186.69 69.85)
+			(xy 213.36 99.06) (xy 199.39 99.06)
 		)
 		(stroke
@@
 	(wire
 		(pts
-			(xy 262.89 80.01) (xy 262.89 77.47)
-		)
-		(stroke
-			(width 0)
-			(type default)
-		)
-	)
-	(wire
-		(pts
 			(xy 229.87 142.24) (xy 224.79 142.24)
 		)
@@
 			(width 0)
 			(type default)
-		)
-	)
-	(label "OUT2_POSITIVE"
-		(at 205.74 74.93 180)
-		(effects
-			(font
-				(size 1.27 1.27)
-			)
-			(justify right bottom)
 		)
 	)
@@
 		)
 	)
-	(label "OUT2_POSITIVE"
-		(at 147.32 58.42 0)
-		(effects
-			(font
-				(size 1.27 1.27)
-			)
-			(justify left bottom)
-		)
-	)
 	(label "SENS1"
 		(at 74.93 78.74 0)
@@
 		)
 	)
-	(label "OUT2_NEGATIVE"
-		(at 147.32 60.96 0)
-		(effects
-			(font
-				(size 1.27 1.27)
-			)
-			(justify left bottom)
-		)
-	)
 	(label "DCF_SIG"
 		(at 147.32 81.28 0)
@@
 			)
 			(justify left bottom)
-		)
-	)
-	(label "OUT2_NEGATIVE"
-		(at 205.74 80.01 180)
-		(effects
-			(font
-				(size 1.27 1.27)
-			)
-			(justify right bottom)
 		)
 	)
@@
 	)
 	(symbol
-		(lib_id "Connector_Generic:Conn_01x02")
-		(at 267.97 74.93 0)
-		(unit 1)
-		(body_style 1)
-		(exclude_from_sim no)
-		(in_bom yes)
-		(on_board yes)
-		(in_pos_files yes)
-		(dnp no)
-		(fields_autoplaced yes)
-		(property "Reference" "J5"
-			(at 270.002 74.9878 0)
-			(show_name no)
-			(do_not_autoplace no)
-			(effects
-				(font
-					(size 1.27 1.27)
-				)
-				(justify left)
-			)
-		)
-		(property "Value" "Conn_01x02"
-			(at 270.002 77.4121 0)
-			(show_name no)
-			(do_not_autoplace no)
-			(effects
-				(font
-					(size 1.27 1.27)
-				)
-				(justify left)
-			)
-		)
-		(property "Footprint" "Connector_JST:JST_XH_S2B-XH-A-1_1x02_P2.50mm_Horizontal"
-			(at 267.97 74.93 0)
-			(hide yes)
-			(show_name no)
-			(do_not_autoplace no)
-			(effects
-				(font
-					(size 1.27 1.27)
-				)
-			)
-		)
-		(property "Datasheet" ""
-			(at 267.97 74.93 0)
-			(hide yes)
-			(show_name no)
-			(do_not_autoplace no)
-			(effects
-				(font
-					(size 1.27 1.27)
-				)
-			)
-		)
-		(property "Description" "Generic connector, single row, 01x02, script generated (kicad-library-utils/schlib/autogen/connector/)"
-			(at 267.97 74.93 0)
-			(hide yes)
-			(show_name no)
-			(do_not_autoplace no)
-			(effects
-				(font
-					(size 1.27 1.27)
-				)
-			)
-		)
-		(pin "1"
-		)
-		(pin "2"
-		)
-		(instances
-			(project "pragotron-clock"
-				(path "/c2785e23-16ef-46a4-bf22-e47ee5f90a07"
-					(reference "J5")
-					(unit 1)
-				)
-			)
-		)
-	)
-	(symbol
 		(lib_id "power:GND")
 		(at 218.44 102.87 0)
@@
 					(unit 1)
 				)
-			)
-		)
-	)
-	(symbol
-		(lib_id "Device:Fuse")
-		(at 246.38 74.93 90)
-		(unit 1)
-		(body_style 1)
-		(exclude_from_sim no)
-		(in_bom yes)
-		(on_board yes)
-		(in_pos_files yes)
-		(dnp no)
-		(fields_autoplaced yes)
-		(property "Reference" "F2"
-			(at 246.38 70.0235 90)
-			(show_name no)
-			(do_not_autoplace no)
-			(effects
-				(font
-					(size 1.27 1.27)
-				)
-			)
-		)
-		(property "Value" "Fuse"
-			(at 246.38 72.4478 90)
-			(show_name no)
-			(do_not_autoplace no)
-			(effects
-				(font
-					(size 1.27 1.27)
-				)
-			)
-		)
-		(property "Footprint" "Fuse:Fuse_1206_3216Metric_Pad1.42x1.75mm_HandSolder"
-			(at 246.38 76.708 90)
-			(hide yes)
-			(show_name no)
-			(do_not_autoplace no)
-			(effects
-				(font
-					(size 1.27 1.27)
-				)
-			)
-		)
-		(property "Datasheet" ""
-			(at 246.38 74.93 0)
-			(hide yes)
-			(show_name no)
-			(do_not_autoplace no)
-			(effects
-				(font
-					(size 1.27 1.27)
-				)
-			)
-		)
-		(property "Description" "Fuse"
-			(at 246.38 74.93 0)
-			(hide yes)
-			(show_name no)
-			(do_not_autoplace no)
-			(effects
-				(font
-					(size 1.27 1.27)
-				)
-			)
-		)
-		(pin "2"
-		)
-		(pin "1"
-		)
-		(instances
-			(project "pragotron-clock"
-				(path "/c2785e23-16ef-46a4-bf22-e47ee5f90a07"
-					(reference "F2")
-					(unit 1)
-				)

Commit message: schematics finished
Parts:
- added C4, C5: 300p, Capacitor_SMD:C_1206_3216Metric_Pad1.33x1.80mm_HandSolder, symbol Device:C
- added L1: 20u, JS_Local:RLS226, symbol Device:L
Connections:
- net +24V: now also L1.1; no longer PS1.2 (+VIN)
- net +5V: now also C5.2
- net GND: now also C4.1, C4.2
- new net: C5.1, L1.2, PS1.2 (+VIN)
Other:
- moved on the sheet: C1

Commit message: pcb
Connections:
- net +24V: now also L1.2; no longer L1.1
- net +5V: now also C5.1; no longer C5.2
- net GND: no longer C1.2, C4.1, J7.2, J7.3, PS1.1 (-VIN)
- new net: C5.2, L1.1, PS1.2 (+VIN)
- new net VIN-: C1.2, C4.1, J7.2, J7.3, PS1.1 (-VIN)
Other:
- note added: "DCF INPUT"
- note added: "POWER SUPPLY"
- moved on the sheet: C1, C4, C5, J6, J7, L1, PS1

Commit message: schematics
Parts:
- added C6: 100n, symbol Device:C
Connections:
- net +3V3: now also C6.1
- net GND: now also C6.2
Other:
- moved on the sheet: J6
Changed lines of the file:
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@@
 	(text "GND"
 		(exclude_from_sim no)
-		(at 131.826 178.054 0)
+		(at 230.886 136.144 0)
 		(effects
 			(font
@@
 	(text "DCF INPUT"
 		(exclude_from_sim no)
-		(at 145.542 156.21 0)
+		(at 244.602 114.3 0)
 		(effects
 			(font
@@
 	(text "SIGNAL"
 		(exclude_from_sim no)
-		(at 130.302 175.514 0)
+		(at 229.362 133.604 0)
 		(effects
 			(font
@@
 	(text "EN"
 		(exclude_from_sim no)
-		(at 132.334 173.228 0)
+		(at 231.394 131.318 0)
 		(effects
 			(font
@@
 	(text "VCC"
 		(exclude_from_sim no)
-		(at 131.826 180.594 0)
+		(at 230.886 138.684 0)
 		(effects
 			(font
@@
 	)
 	(junction
-		(at 158.75 177.8)
-		(diameter 0)
-		(color 0 0 0 0)
-	)
-	(junction
 		(at 160.02 111.76)
 		(diameter 0)
@@
 	)
 	(junction
+		(at 260.35 138.43)
+		(diameter 0)
+		(color 0 0 0 0)
+	)
+	(junction
 		(at 40.64 148.59)
 		(diameter 0)
@@
 	(junction
 		(at 97.79 148.59)
+		(diameter 0)
+		(color 0 0 0 0)
+	)
+	(junction
+		(at 257.81 151.13)
+		(diameter 0)
+		(color 0 0 0 0)
+	)
+	(junction
+		(at 257.81 135.89)
 		(diameter 0)
 		(color 0 0 0 0)
@@
 	(wire
 		(pts
-			(xy 140.97 172.72) (xy 158.75 172.72)
+			(xy 240.03 130.81) (xy 257.81 130.81)
 		)
 		(stroke
@@
 	(wire
 		(pts
-			(xy 161.29 168.91) (xy 161.29 180.34)
+			(xy 257.81 151.13) (xy 269.24 151.13)
+		)
+		(stroke
+			(width 0)
+			(type default)
+		)
+	)
+	(wire
+		(pts
+			(xy 269.24 138.43) (xy 260.35 138.43)
+		)
+		(stroke
+			(width 0)
+			(type default)
+		)
+	)
+	(wire
+		(pts
+			(xy 260.35 127) (xy 260.35 138.43)
 		)
 		(stroke
@@
 	(wire
 		(pts
-			(xy 140.97 177.8) (xy 158.75 177.8)
+			(xy 240.03 135.89) (xy 257.81 135.89)
 		)
 		(stroke
@@
 	(wire
 		(pts
+			(xy 257.81 151.13) (xy 257.81 153.67)
+		)
+		(stroke
+			(width 0)
+			(type default)
+		)
+	)
+	(wire
+		(pts
 			(xy 220.98 99.06) (xy 220.98 95.25)
 		)
@@
 	(wire
 		(pts
-			(xy 140.97 180.34) (xy 161.29 180.34)
+			(xy 240.03 138.43) (xy 260.35 138.43)
 		)
 		(stroke
@@
 	(wire
 		(pts
-			(xy 158.75 177.8) (xy 158.75 185.42)
+			(xy 257.81 135.89) (xy 257.81 151.13)
 		)
 		(stroke
@@
 	(wire
 		(pts
-			(xy 158.75 172.72) (xy 158.75 177.8)
+			(xy 257.81 130.81) (xy 257.81 135.89)
 		)
 		(stroke
@@
 	(wire
 		(pts
-			(xy 140.97 175.26) (xy 163.83 175.26)
+			(xy 240.03 133.35) (xy 262.89 133.35)
 		)
 		(stroke
@@
 	(wire
 		(pts
+			(xy 269.24 140.97) (xy 269.24 138.43)
+		)
+		(stroke
+			(width 0)
+			(type default)
+		)
+	)
+	(wire
+		(pts
 			(xy 69.85 175.26) (xy 77.47 175.26)
+		)
+		(stroke
+			(width 0)
+			(type default)
+		)
+	)
+	(wire
+		(pts
+			(xy 269.24 151.13) (xy 269.24 148.59)
 		)
 		(stroke
@@
 	)
 	(label "DCF_SIG"
-		(at 163.83 175.26 0)
+		(at 262.89 133.35 0)
 		(effects
 			(font
@@
 	(symbol
 		(lib_id "power:+3V3")
-		(at 161.29 168.91 0)
+		(at 260.35 127 0)
 		(unit 1)
 		(body_style 1)
@@
 		(fields_autoplaced yes)
 		(property "Reference" "#PWR08"
-			(at 161.29 172.72 0)
+			(at 260.35 130.81 0)
 			(hide yes)
 			(show_name no)
@@
 		)
 		(property "Value" "+3V3"
-			(at 161.29 164.7769 0)
+			(at 260.35 122.8669 0)
 			(show_name no)
 			(do_not_autoplace no)
@@
 		)
 		(property "Footprint" ""
-			(at 161.29 168.91 0)
+			(at 260.35 127 0)
 			(hide yes)
 			(show_name no)
@@
 		)
 		(property "Datasheet" ""
-			(at 161.29 168.91 0)
+			(at 260.35 127 0)
 			(hide yes)
 			(show_name no)
@@
 		)
 		(property "Description" "Power symbol creates a global label with name \"+3V3\""
-			(at 161.29 168.91 0)
+			(at 260.35 127 0)
 			(hide yes)
 			(show_name no)
@@
 	)
 	(symbol
+		(lib_id "Device:C")
+		(at 269.24 144.78 0)
+		(unit 1)
+		(body_style 1)
+		(exclude_from_sim no)
+		(in_bom yes)
+		(on_board yes)
+		(in_pos_files yes)
+		(dnp no)
+		(fields_autoplaced yes)
+		(property "Reference" "C6"
+			(at 273.05 143.5099 0)
+			(show_name no)
+			(do_not_autoplace no)
+			(effects
+				(font
+					(size 1.27 1.27)
+				)
+				(justify left)
+			)
+		)
+		(property "Value" "100n"
+			(at 273.05 146.0499 0)
+			(show_name no)
+			(do_not_autoplace no)
+			(effects
+				(font
+					(size 1.27 1.27)
+				)
+				(justify left)
+			)
+		)
+		(property "Footprint" ""
+			(at 270.2052 148.59 0)
+			(hide yes)
+			(show_name no)
+			(do_not_autoplace no)
+			(effects
+				(font
+					(size 1.27 1.27)
+				)
+			)
+		)
+		(property "Datasheet" ""
+			(at 269.24 144.78 0)
+			(hide yes)
+			(show_name no)
+			(do_not_autoplace no)
+			(effects
+				(font
+					(size 1.27 1.27)
+				)
+			)
+		)
+		(property "Description" "Unpolarized capacitor"
+			(at 269.24 144.78 0)
+			(hide yes)
+			(show_name no)
+			(do_not_autoplace no)
+			(effects
+				(font
+					(size 1.27 1.27)
+				)
+			)
+		)
+		(pin "2"
+		)
+		(pin "1"
+		)
+		(instances
+			(project "pragotron-clock"
+				(path "/c2785e23-16ef-46a4-bf22-e47ee5f90a07"
+					(reference "C6")
+					(unit 1)
+				)
+			)
+		)
+	)
+	(symbol
 		(lib_id "Device:Fuse")
 		(at 246.38 59.69 90)
@@
 	(symbol
 		(lib_id "Connector_Generic:Conn_01x04")
-		(at 135.89 177.8 180)
+		(at 234.95 135.89 180)
 		(unit 1)
 		(body_style 1)
@@
 		(fields_autoplaced yes)
 		(property "Reference" "J6"
-			(at 135.89 167.3055 0)
+			(at 234.95 125.3955 0)
 			(show_name no)
 			(do_not_autoplace no)
@@
 		)
 		(property "Value" "Conn_01x04"
-			(at 135.89 169.7298 0)
+			(at 234.95 127.8198 0)
 			(show_name no)
 			(do_not_autoplace no)
@@
 		)
 		(property "Footprint" "JS_Local:DCF77"
-			(at 135.89 177.8 0)
+			(at 234.95 135.89 0)
 			(hide yes)
 			(show_name no)
@@
 		)
 		(property "Datasheet" ""
-			(at 135.89 177.8 0)
+			(at 234.95 135.89 0)
 			(hide yes)
 			(show_name no)
@@
 		)
 		(property "Description" "Generic connector, single row, 01x04, script generated (kicad-library-utils/schlib/autogen/connector/)"
-			(at 135.89 177.8 0)
+			(at 234.95 135.89 0)
 			(hide yes)
 			(show_name no)
@@
 	(symbol
 		(lib_id "power:GND")
-		(at 158.75 185.42 0)
+		(at 257.81 153.67 0)
 		(unit 1)
 		(body_style 1)
@@
 		(fields_autoplaced yes)
 		(property "Reference" "#PWR07"
-			(at 158.75 191.77 0)
+			(at 257.81 160.02 0)
 			(hide yes)
 			(show_name no)
@@
 		)
 		(property "Value" "GND"
-			(at 158.75 189.5531 0)
+			(at 257.81 157.8031 0)
 			(show_name no)
 			(do_not_autoplace no)
@@
 		)
 		(property "Footprint" ""
-			(at 158.75 185.42 0)
+			(at 257.81 153.67 0)
 			(hide yes)
 			(show_name no)
@@
 		)
 		(property "Datasheet" ""
-			(at 158.75 185.42 0)
+			(at 257.81 153.67 0)
 			(hide yes)
 			(show_name no)
@@
 		)
 		(property "Description" "Power symbol creates a global label with name \"GND\" , ground"
-			(at 158.75 185.42 0)
-			(hide yes)
-			(show_name no)
+			(at 257.81 153.67 0)
+			(hide yes)
+			(show_name no)

Commit message: gerber v1.0
Parts:
- C6: footprint (none) -> Capacitor_SMD:C_1206_3216Metric_Pad1.33x1.80mm_HandSolder
Changed lines of the file:
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@@
 			)
 		)
-		(property "Footprint" ""
+		(property "Footprint" "Capacitor_SMD:C_1206_3216Metric_Pad1.33x1.80mm_HandSolder"
 			(at 270.2052 148.59 0)
 			(hide yes)
