File: pcb/pragotron-clock.kicad_sch (KiCad schematic)
At the start: 18 parts, among them J1 Conn_01x02, J2 Conn_01x03, J3 Conn_01x03, J6 Conn_01x04, J7 694108301002, U1 L293D

Commit message: fuse specification
Parts:
- F1: value Fuse -> 200mA T
Changed lines of the file:
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@@
 		(fields_autoplaced yes)
 		(property "Reference" "F1"
-			(at 246.38 54.7835 90)
+			(at 246.38 53.34 90)
 			(show_name no)
 			(do_not_autoplace no)
@@
 			)
 		)
-		(property "Value" "Fuse"
-			(at 246.38 57.2078 90)
+		(property "Value" "200mA T"
+			(at 246.38 55.88 90)
 			(show_name no)
 			(do_not_autoplace no)
