File: pcb/pragotron-clock.kicad_sch (KiCad schematic)
At the start: 18 parts, among them J1 Conn_01x02, J2 Conn_01x03, J3 Conn_01x03, J6 Conn_01x04, J7 694108301002, U1 L293D

Commit message: remove ground separation, turn around esp8266
Parts:
- removed C4: 300p, Capacitor_SMD:C_1206_3216Metric_Pad1.33x1.80mm_HandSolder, symbol Device:C
Connections:
- net VIN- is gone; now on net GND: C1.2, J7.2, J7.3, PS1.1 (-VIN)
Changed lines of the file:
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@@
 	)
 	(junction
-		(at 69.85 177.8)
-		(diameter 0)
-		(color 0 0 0 0)
-	)
-	(junction
 		(at 138.43 46.99)
 		(diameter 0)
@@
 	)
 	(junction
+		(at 74.93 177.8)
+		(diameter 0)
+		(color 0 0 0 0)
+	)
+	(junction
 		(at 187.96 111.76)
 		(diameter 0)
@@
 	)
 	(junction
-		(at 87.63 177.8)
+		(at 80.01 177.8)
 		(diameter 0)
 		(color 0 0 0 0)
@@
 	(wire
 		(pts
-			(xy 74.93 181.61) (xy 69.85 181.61)
-		)
-		(stroke
-			(width 0)
-			(type default)
-		)
-	)
-	(wire
-		(pts
 			(xy 63.5 83.82) (xy 72.39 83.82)
 		)
@@
 	(wire
 		(pts
-			(xy 69.85 181.61) (xy 69.85 177.8)
-		)
-		(stroke
-			(width 0)
-			(type default)
-		)
-	)
-	(wire
-		(pts
 			(xy 85.09 46.99) (xy 92.71 46.99)
 		)
@@
 	(wire
 		(pts
-			(xy 69.85 177.8) (xy 74.93 177.8)
-		)
-		(stroke
-			(width 0)
-			(type default)
-		)
-	)
-	(wire
-		(pts
 			(xy 109.22 81.28) (xy 109.22 91.44)
 		)
@@
 	(wire
 		(pts
-			(xy 82.55 181.61) (xy 87.63 181.61)
-		)
-		(stroke
-			(width 0)
-			(type default)
-		)
-	)
-	(wire
-		(pts
 			(xy 257.81 130.81) (xy 257.81 135.89)
 		)
@@
 	(wire
 		(pts
-			(xy 87.63 181.61) (xy 87.63 177.8)
-		)
-		(stroke
-			(width 0)
-			(type default)
-		)
-	)
-	(wire
-		(pts
 			(xy 186.69 69.85) (xy 205.74 69.85)
 		)
@@
 	(wire
 		(pts
-			(xy 80.01 177.8) (xy 87.63 177.8)
+			(xy 80.01 177.8) (xy 106.68 177.8)
 		)
 		(stroke
@@
 	(wire
 		(pts
-			(xy 87.63 177.8) (xy 106.68 177.8)
-		)
-		(stroke
-			(width 0)
-			(type default)
-		)
-	)
-	(wire
-		(pts
-			(xy 50.8 177.8) (xy 69.85 177.8)
+			(xy 50.8 177.8) (xy 74.93 177.8)
 		)
 		(stroke
@@
 	(wire
 		(pts
+			(xy 74.93 177.8) (xy 80.01 177.8)
+		)
+		(stroke
+			(width 0)
+			(type default)
+		)
+	)
+	(wire
+		(pts
 			(xy 269.24 140.97) (xy 269.24 138.43)
 		)
@@
 					(unit 1)
 				)
-			)
-		)
-	)
-	(symbol
-		(lib_id "Device:C")
-		(at 78.74 181.61 90)
-		(unit 1)
-		(body_style 1)
-		(exclude_from_sim no)
-		(in_bom yes)
-		(on_board yes)
-		(in_pos_files yes)
-		(dnp no)
-		(property "Reference" "C4"
-			(at 78.74 185.928 90)
-			(show_name no)
-			(do_not_autoplace no)
-			(effects
-				(font
-					(size 1.27 1.27)
-				)
-			)
-		)
-		(property "Value" "300p"
-			(at 78.74 188.976 90)
-			(show_name no)
-			(do_not_autoplace no)
-			(effects
-				(font
-					(size 1.27 1.27)
-				)
-			)
-		)
-		(property "Footprint" "Capacitor_SMD:C_1206_3216Metric_Pad1.33x1.80mm_HandSolder"
-			(at 82.55 180.6448 0)
-			(hide yes)
-			(show_name no)
-			(do_not_autoplace no)
-			(effects
-				(font
-					(size 1.27 1.27)
-				)
-			)
-		)
-		(property "Datasheet" ""
-			(at 78.74 181.61 0)
-			(hide yes)
-			(show_name no)
-			(do_not_autoplace no)
-			(effects
-				(font
-					(size 1.27 1.27)
-				)
-			)
-		)
-		(property "Description" "Unpolarized capacitor"
-			(at 78.74 181.61 0)
-			(hide yes)
-			(show_name no)
-			(do_not_autoplace no)
-			(effects
-				(font
-					(size 1.27 1.27)
-				)
-			)
-		)
-		(pin "2"
-		)
-		(pin "1"
-		)
-		(instances
-			(project "pragotron-clock"
-				(path "/c2785e23-16ef-46a4-bf22-e47ee5f90a07"
-					(reference "C4")
-					(unit 1)
-				)
